File: Hardware/Optical_Tracking_Odometry_Sensor.kicad_pcb (KiCad board)
At the start: 2 copper layers, 25.4 x 25.4 mm, 55 parts, among them J3 CONN_06NO_SILK_NO_POP, Q1 100mA/20V/3.8Ω, Q2 100mA/20V/3.8Ω, U1 PAA5160E1-Q, U2 LSM6DS0, U3 STM32C011F6U6, U4 RT9080-18GJ5

Commit message: Improvements
Parts:
- moved J3 0.43 mm to (142.2, 116.0)
- moved FD1 0.27 mm to (141.1, 95.0)
- moved FD2 0.27 mm to (141.1, 95.0)
- moved FD3 0.27 mm to (158.5, 112.4)
- moved FD4 0.27 mm to (158.5, 112.4)
- moved H2 0.23 mm to (138.5, 95.0)
- moved H3 0.23 mm to (158.5, 95.0)
- moved H1 0.23 mm to (138.5, 115.0)
- moved H4 0.23 mm to (158.5, 115.0)
Routing:
- net 3.3V: track 79.3 -> 78.7 mm
- net GND: vias 42 -> 41
Other:
- board size 25.4 x 25.4 mm -> 25 x 25 mm

Commit message: Good
Parts:
- removed U$20: , Optical_Tracking_Odometry_Sensor:#PWR#0
- removed U$25: , Optical_Tracking_Odometry_Sensor:PWR0
- removed U$26: , Optical_Tracking_Odometry_Sensor:#I2C#0
- added REF**: logo, Optical_Tracking_Odometry_Sensor:logo, F.Cu at (156.9, 106.5)
- added kibuzzard-6857E631: G***, kibuzzard-6857E631, F.Cu at (138.3, 98.0)
- added kibuzzard-6857E6C8: G***, kibuzzard-6857E6C8, F.Cu at (138.3, 106.7)
- added kibuzzard-6857E9FE: G***, kibuzzard-6857E9FE, B.Cu at (137.7, 104.8)
- added kibuzzard-6857EA13: G***, kibuzzard-6857EA13, B.Cu at (159.5, 103.6)
- added kibuzzard-6857EA7B: G***, kibuzzard-6857EA7B, B.Cu at (142.1, 113.5)
- added kibuzzard-6857EA92: G***, kibuzzard-6857EA92, B.Cu at (144.7, 113.5)
- added kibuzzard-6857EA9A: G***, kibuzzard-6857EA9A, B.Cu at (147.2, 113.5)
- added kibuzzard-6857EAA2: G***, kibuzzard-6857EAA2, B.Cu at (149.8, 113.5)
- added kibuzzard-6857EAAB: G***, kibuzzard-6857EAAB, B.Cu at (152.3, 113.5)
- added kibuzzard-6857EAE5: G***, kibuzzard-6857EAE5, F.Cu at (142.1, 113.5)
- added kibuzzard-6857EAF6: G***, kibuzzard-6857EAF6, F.Cu at (144.7, 113.5)
- added kibuzzard-6857EAFE: G***, kibuzzard-6857EAFE, F.Cu at (147.2, 113.5)
- added kibuzzard-6857EB06: G***, kibuzzard-6857EB06, F.Cu at (149.8, 113.5)
- added kibuzzard-6857EB0C: G***, kibuzzard-6857EB0C, F.Cu at (152.3, 113.5)
- added kibuzzard-6857EB13: G***, kibuzzard-6857EB13, F.Cu at (154.8, 113.5)
- added kibuzzard-6857EB25: G***, kibuzzard-6857EB25, B.Cu at (154.8, 113.5)
Connections:
- net /STM_IO10 renamed /DBG_RX
- net /STM_IO9 renamed /DBG_TX
