File: Hardware/Optical_Tracking_Odometry_Sensor.kicad_pcb (KiCad board)
At the start: 2 copper layers, 25 x 25 mm, 61 parts, among them J3 CONN_06NO_SILK_NO_POP, Q1 100mA/20V/3.8Ω, Q2 100mA/20V/3.8Ω, U1 PAA5160E1-Q, U2 LSM6DS0, U3 STM32C011F6U6, U4 RT9080-18GJ5

Commit message: Updated PCB and Readme
Parts:
- U1: value PAA5160E1-Q -> PAA5163E1-Q; footprint Optical_Tracking_Odometry_Sensor:PAA5160E1-Q -> Optical_Tracking_Odometry_Sensor:PAA5163E1-Q

Commit message: Updated cad with 3d model
Parts:
- C1, C10, C11, C12, C13, C14, C2, C3, C4, C5, C6, C7, C8, C9: footprint Optical_Tracking_Odometry_Sensor:0603 -> Capacitor_SMD:C_0603_1608Metric
- D1: footprint Optical_Tracking_Odometry_Sensor:LED-0603 -> LED_SMD:LED_0603_1608Metric
- D2, D3, D4: footprint Optical_Tracking_Odometry_Sensor:0603 -> Diode_SMD:D_0603_1608Metric
- Q1, Q2: footprint Optical_Tracking_Odometry_Sensor:SOT-416FL -> Package_TO_SOT_SMD:SOT-416
- R1, R2, R3, R4, R5, R6, R7: footprint Optical_Tracking_Odometry_Sensor:0603 -> Resistor_SMD:R_0603_1608Metric
- U2: footprint Optical_Tracking_Odometry_Sensor:LGA14L -> Package_LGA:LGA-14_3x2.5mm_P0.5mm_LayoutBorder3x4y
- U3: footprint Optical_Tracking_Odometry_Sensor:STM32C011F6U6 -> Package_DFN_QFN:ST_UFQFPN-20_3x3mm_P0.5mm
- U4: footprint Optical_Tracking_Odometry_Sensor:SOT23-5 -> Package_TO_SOT_SMD:SOT-23-5
- moved Q2 0.57 mm to (145.9, 109.6), turned to 180 degrees
- moved Q1 0.55 mm to (142.7, 99.2), turned to 90 degrees
- moved U4 0.06 mm to (143.4, 107.6), turned to 90 degrees
- turned D1 to 0 degrees
Connections:
- R1 pad 2: Net-(D1-PadA) -> Net-(D1-A)
Routing:
- net Net-(D1-PadA): track 2.37 -> 0.00 mm, vias 1 -> 0
- net Net-(D1-A): track 0.00 -> 2.37 mm, vias 0 -> 1
