File: Hardware/Optical_Tracking_Odometry_Sensor.kicad_sch (KiCad schematic)
At the start: 35 parts, among them J3 CONN_06NO_SILK_NO_POP, Q1 100mA/20V/3.8Ω, Q2 100mA/20V/3.8Ω, U1 PAA5160E1-Q, U2 LSM6DS0, U3 STM32C011F6U6, U4 RT9080-18GJ5

Commit message: Good
Connections:
- net STM_IO10 renamed DBG_RX
- net STM_IO9 renamed DBG_TX
Changed lines of the file:
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@@
 		)
 	)
-	(label "STM_IO9"
+	(label "DBG_TX"
 		(at 63.5 60.96 180)
 		(effects
@@
 		)
 	)
-	(label "STM_IO10"
+	(label "DBG_RX"
 		(at 63.5 63.5 180)
 		(effects
@@
 		)
 	)
-	(label "STM_IO10"
+	(label "DBG_RX"
 		(at 236.22 81.28 0)
 		(effects
@@
 		)
 	)
-	(label "STM_IO9"
+	(label "DBG_TX"
 		(at 236.22 83.82 0)
 		(effects
