File: Hardware/Optical_Tracking_Odometry_Sensor.kicad_sch (KiCad schematic)
At the start: 35 parts, among them J3 CONN_06NO_SILK_NO_POP, Q1 100mA/20V/3.8Ω, Q2 100mA/20V/3.8Ω, U1 PAA5160E1-Q, U2 LSM6DS0, U3 STM32C011F6U6, U4 RT9080-18GJ5

Commit message: Updated PCB and Readme
Parts:
- U1: value PAA5160E1-Q -> PAA5163E1-Q; footprint Optical_Tracking_Odometry_Sensor:PAA5160E1-Q -> Optical_Tracking_Odometry_Sensor:PAA5163E1-Q; symbol Optical_Tracking_Odometry_Sensor-eagle-import:PAA5160E1-Q -> Optical_Tracking_Odometry_Sensor-eagle-import:PAA5163E1-Q
Other:
- note added: "Optical Tracking Sensor - PAA5163E1-QV22"
- note added: "PAA5163 Power Control and Regulator - RT9080"
- note removed: "LSM6DSV ?"
- note removed: "Optical Tracking Sensor - PAA5160E1-Q"
- note removed: "PAA5160 Power Control and Regulator - RT9080"
- note removed: "PAA5163E1 ?"

Commit message: Updated cad with 3d model
Parts:
- C1, C10, C11, C12, C13, C14, C2, C3, C4, C5, C6, C7, C8, C9: footprint Optical_Tracking_Odometry_Sensor:0603 -> Capacitor_SMD:C_0603_1608Metric
- D1: footprint Optical_Tracking_Odometry_Sensor:LED-0603 -> LED_SMD:LED_0603_1608Metric; symbol Optical_Tracking_Odometry_Sensor-eagle-import:LED-RED_0603-KB -> Device:LED
- D2, D3, D4: footprint Optical_Tracking_Odometry_Sensor:0603 -> Diode_SMD:D_0603_1608Metric
- I2C0, J3, PWR0, U$1: now left out of the parts list
- Q1, Q2: footprint Optical_Tracking_Odometry_Sensor:SOT-416FL -> Package_TO_SOT_SMD:SOT-416
- R1, R2, R3, R4, R5, R6, R7: footprint Optical_Tracking_Odometry_Sensor:0603 -> Resistor_SMD:R_0603_1608Metric
- U2: footprint Optical_Tracking_Odometry_Sensor:LGA14L -> Package_LGA:LGA-14_3x2.5mm_P0.5mm_LayoutBorder3x4y
- U3: footprint Optical_Tracking_Odometry_Sensor:STM32C011F6U6 -> Package_DFN_QFN:ST_UFQFPN-20_3x3mm_P0.5mm
- U4: footprint Optical_Tracking_Odometry_Sensor:SOT23-5 -> Package_TO_SOT_SMD:SOT-23-5
Connections:
- net GND: now also D1.1 (K); no longer D1.C
- net at R1.2: now also D1.2 (A); no longer D1.A
Changed lines of the file:
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@@
 	(wire
 		(pts
-			(xy 176.53 116.84) (xy 176.53 111.76)
-		)
-		(stroke
-			(width 0.1524)
-			(type solid)
-		)
-	)
-	(wire
-		(pts
 			(xy 256.54 35.56) (xy 256.54 38.1)
 		)
@@
 	(wire
 		(pts
+			(xy 176.53 111.76) (xy 176.53 116.84)
+		)
+		(stroke
+			(width 0)
+			(type default)
+		)
+	)
+	(wire
+		(pts
 			(xy 166.37 114.3) (xy 166.37 111.76)
 		)
@@
 			)
 		)
-		(property "Footprint" "Optical_Tracking_Odometry_Sensor:0603"
+		(property "Footprint" "Diode_SMD:D_0603_1608Metric"
 			(at 179.07 83.82 0)
 			(effects
@@
 			)
 		)
-		(property "Footprint" "Optical_Tracking_Odometry_Sensor:0603"
+		(property "Footprint" "Resistor_SMD:R_0603_1608Metric"
 			(at 166.37 119.38 0)
 			(effects
@@
 			)
 		)
-		(property "Footprint" "Optical_Tracking_Odometry_Sensor:0603"
+		(property "Footprint" "Capacitor_SMD:C_0603_1608Metric"
 			(at 60.96 193.04 0)
 			(effects
@@
 			)
 		)
-		(property "Footprint" "Optical_Tracking_Odometry_Sensor:0603"
+		(property "Footprint" "Diode_SMD:D_0603_1608Metric"
 			(at 153.67 83.82 0)
 			(effects
@@
 	)
 	(symbol
-		(lib_id "Optical_Tracking_Odometry_Sensor-eagle-import:LED-RED_0603-KB")
-		(at 176.53 119.38 0)
+		(lib_id "Device:LED")
+		(at 176.53 120.65 90)
 		(unit 1)
 		(exclude_from_sim no)
@@
 		(dnp no)
 		(property "Reference" "D1"
-			(at 173.101 123.952 90)
+			(at 174.498 122.428 0)
 			(effects
 				(font
@@
 		)
 		(property "Value" "Blue"
-			(at 178.435 123.952 90)
+			(at 178.816 123.19 0)
 			(effects
 				(font
@@
 			)
 		)
-		(property "Footprint" "Optical_Tracking_Odometry_Sensor:LED-0603"
-			(at 176.53 119.38 0)
+		(property "Footprint" "LED_SMD:LED_0603_1608Metric"
+			(at 176.53 120.65 0)
 			(effects
 				(font
@@
 			)
 		)
-		(property "Datasheet" ""
-			(at 176.53 119.38 0)
+		(property "Datasheet" "~"
+			(at 176.53 120.65 0)
 			(effects
 				(font
@@
 			)
 		)
-		(property "Description" ""
-			(at 176.53 119.38 0)
+		(property "Description" "Light emitting diode"
+			(at 176.53 120.65 0)
 			(effects
 				(font
@@
 			)
 		)
-		(pin "C"
+		(property "Sim.Pins" "1=K 2=A"
+			(at 176.53 120.65 0)
+			(effects
+				(font
+					(size 1.27 1.27)
+				)
+				(hide yes)
+			)
 		)
-		(pin "A"
+		(pin "1"
+		)
+		(pin "2"
 		)
 		(instances
@@
 			)
 		)
-		(property "Footprint" "Optical_Tracking_Odometry_Sensor:0603"
+		(property "Footprint" "Capacitor_SMD:C_0603_1608Metric"
 			(at 256.54 45.72 0)
 			(effects
@@
 			)
 		)
-		(property "Footprint" "Optical_Tracking_Odometry_Sensor:0603"
+		(property "Footprint" "Resistor_SMD:R_0603_1608Metric"
 			(at 231.14 45.72 0)
 			(effects
@@
 			)
 		)
-		(property "Footprint" "Optical_Tracking_Odometry_Sensor:0603"
+		(property "Footprint" "Capacitor_SMD:C_0603_1608Metric"
 			(at 195.58 45.72 0)
 			(effects
@@
 			)
 		)
-		(property "Footprint" "Optical_Tracking_Odometry_Sensor:0603"
+		(property "Footprint" "Resistor_SMD:R_0603_1608Metric"
 			(at 143.51 184.15 0)
 			(effects
@@
 			)
 		)
-		(property "Footprint" "Optical_Tracking_Odometry_Sensor:SOT-416FL"
+		(property "Footprint" "Package_TO_SOT_SMD:SOT-416"
 			(at 238.76 40.64 0)
 			(effects
@@
 			)
 		)
-		(property "Footprint" "Optical_Tracking_Odometry_Sensor:0603"
+		(property "Footprint" "Capacitor_SMD:C_0603_1608Metric"
 			(at 45.72 193.04 0)
 			(effects
@@
 			)
 		)
-		(property "Footprint" "Optical_Tracking_Odometry_Sensor:LGA14L"
+		(property "Footprint" "Package_LGA:LGA-14_3x2.5mm_P0.5mm_LayoutBorder3x4y"
 			(at 83.82 124.46 0)
 			(effects
@@
 			)
 		)
-		(property "Footprint" "Optical_Tracking_Odometry_Sensor:0603"
+		(property "Footprint" "Resistor_SMD:R_0603_1608Metric"
 			(at 158.75 184.15 0)
 			(effects
@@
 			)
 		)
-		(property "Footprint" "Optical_Tracking_Odometry_Sensor:0603"
+		(property "Footprint" "Resistor_SMD:R_0603_1608Metric"
 			(at 142.24 45.72 0)
 			(effects
@@
 		(unit 1)
 		(exclude_from_sim no)
-		(in_bom yes)
+		(in_bom no)
 		(on_board yes)
 		(dnp no)
@@
 			)
 		)
-		(property "Footprint" "Optical_Tracking_Odometry_Sensor:SOT-416FL"
+		(property "Footprint" "Package_TO_SOT_SMD:SOT-416"
 			(at 149.86 40.64 0)
 			(effects
@@
 			)
 		)
-		(property "Footprint" "Optical_Tracking_Odometry_Sensor:0603"
+		(property "Footprint" "Diode_SMD:D_0603_1608Metric"
 			(at 166.37 83.82 0)
 			(effects
@@
 			)
 		)
-		(property "Footprint" "Optical_Tracking_Odometry_Sensor:0603"
+		(property "Footprint" "Capacitor_SMD:C_0603_1608Metric"
 			(at 43.18 73.66 0)
 			(effects
@@
 			)
 		)
-		(property "Footprint" "Optical_Tracking_Odometry_Sensor:STM32C011F6U6"
+		(property "Footprint" "Package_DFN_QFN:ST_UFQFPN-20_3x3mm_P0.5mm"
 			(at 86.36 60.96 0)
 			(effects
@@
 		(unit 1)
 		(exclude_from_sim no)
-		(in_bom yes)
+		(in_bom no)
 		(on_board yes)
 		(dnp no)
@@
 			)
 		)
-		(property "Footprint" "Optical_Tracking_Odometry_Sensor:SOT23-5"
+		(property "Footprint" "Package_TO_SOT_SMD:SOT-23-5"
 			(at 180.34 43.18 0)
 			(effects
@@
 			)
 		)
-		(property "Footprint" "Optical_Tracking_Odometry_Sensor:0603"
+		(property "Footprint" "Resistor_SMD:R_0603_1608Metric"
 			(at 109.22 38.1 0)
 			(effects
@@
 			)
 		)
-		(property "Footprint" "Optical_Tracking_Odometry_Sensor:0603"
+		(property "Footprint" "Capacitor_SMD:C_0603_1608Metric"
 			(at 27.94 73.66 0)
 			(effects
@@
 			)
 		)
-		(property "Footprint" "Optical_Tracking_Odometry_Sensor:0603"
+		(property "Footprint" "Capacitor_SMD:C_0603_1608Metric"
 			(at 48.26 129.54 0)
 			(effects
@@
 			)
 		)
-		(property "Footprint" "Optical_Tracking_Odometry_Sensor:0603"
+		(property "Footprint" "Capacitor_SMD:C_0603_1608Metric"
 			(at 38.1 193.04 0)
 			(effects
@@
 			)
 		)
-		(property "Footprint" "Optical_Tracking_Odometry_Sensor:0603"
+		(property "Footprint" "Capacitor_SMD:C_0603_1608Metric"
 			(at 109.22 200.66 0)
 			(effects
@@
 			)
 		)
-		(property "Footprint" "Optical_Tracking_Odometry_Sensor:0603"
+		(property "Footprint" "Capacitor_SMD:C_0603_1608Metric"
 			(at 30.48 193.04 0)
 			(effects
@@
 			)
 		)
-		(property "Footprint" "Optical_Tracking_Odometry_Sensor:0603"
+		(property "Footprint" "Capacitor_SMD:C_0603_1608Metric"
 			(at 53.34 193.04 0)
 			(effects
@@
 		(unit 1)
 		(exclude_from_sim no)
-		(in_bom yes)
+		(in_bom no)
 		(on_board yes)
 		(dnp no)
@@
 		(unit 1)
 		(exclude_from_sim no)
-		(in_bom yes)
+		(in_bom no)
 		(on_board yes)
 		(dnp no)
@@
 			)
 		)
-		(property "Footprint" "Optical_Tracking_Odometry_Sensor:0603"
+		(property "Footprint" "Capacitor_SMD:C_0603_1608Metric"
 			(at 35.56 73.66 0)
 			(effects
@@
 			)
 		)
-		(property "Footprint" "Optical_Tracking_Odometry_Sensor:0603"
+		(property "Footprint" "Capacitor_SMD:C_0603_1608Metric"
 			(at 157.48 45.72 0)
 			(effects
@@
 			)
 		)
-		(property "Footprint" "Optical_Tracking_Odometry_Sensor:0603"
+		(property "Footprint" "Resistor_SMD:R_0603_1608Metric"
 			(at 50.8 71.12 0)
 			(effects
@@
 			)
 		)
-		(property "Footprint" "Optical_Tracking_Odometry_Sensor:0603"
+		(property "Footprint" "Capacitor_SMD:C_0603_1608Metric"
 			(at 35.56 129.54 0)
 			(effects
